File: picoSCSI/picoSCSI.kicad_sch (KiCad schematic)
At the start: 19 parts, among them J1 SCSI_CONN, J2 Micro_SD_Card, J3 Floppy Power

Commit message: Start PCB
Parts:
- D1: footprint (none) -> LED_THT:LED_D5.0mm
- D2, D3: value D -> 1N4001; footprint (none) -> Diode_THT:D_DO-41_SOD81_P7.62mm_Horizontal
- H1, H2, H3, H4: footprint (none) -> MountingHole:MountingHole_3.2mm_M3_ISO7380
- J1: footprint (none) -> Connector_IDC:IDC-Header_2x25_P2.54mm_Vertical
- J2: footprint (none) -> Connector_Card:microSD_HC_Wuerth_693072010801
- J3: footprint (none) -> Connector_JST:JST_PH_B4B-PH-K_1x04_P2.00mm_Vertical
- JP1, JP4: footprint (none) -> Connector_PinSocket_2.54mm:PinSocket_1x02_P2.54mm_Vertical
- JP3: footprint (none) -> Jumper:SolderJumper-2_P1.3mm_Open_RoundedPad1.0x1.5mm
- R1: footprint (none) -> Resistor_THT:R_Axial_DIN0204_L3.6mm_D1.6mm_P5.08mm_Horizontal
Connections:
- net SCSI_ACK: now also A1.14 (GPIO10); no longer A1.15 (GPIO11)
- net SCSI_BSY: now also A1.26 (GPIO20); no longer A1.14 (GPIO10)
- net SCSI_CD: now also A1.24 (GPIO18); no longer A1.20 (GPIO15)
- net SCSI_IO: now also A1.29 (GPIO22); no longer A1.21 (GPIO16)
- net SCSI_MSG: now also A1.21 (GPIO16); no longer A1.17 (GPIO13)
- net SCSI_RST: now also A1.27 (GPIO21); no longer A1.16 (GPIO12)
- net SCSI_SEL: now also A1.25 (GPIO19); no longer A1.19 (GPIO14)
- net SD_CLK: now also A1.31 (GPIO26_ADC0)
- net SD_CMD: now also A1.15 (GPIO11)
- net SD_DATA0: now also A1.17 (GPIO13)
- net SD_DATA1: now also A1.16 (GPIO12)
- net SD_DATA2: now also A1.20 (GPIO15)
- net SD_DATA3: now also A1.19 (GPIO14)
- no-connect marks 16 -> 10
