File: picoSCSI/picoSCSI.kicad_pcb (KiCad board)
At the start: 2 copper layers, 60 x 100 mm, 19 parts, among them J1 SCSI_CONN, J2 Micro_SD_Card, J3 Floppy Power

Commit message: tmp
Parts:
- moved H1 105.2 mm to (110.0, 113.8)
- moved J1 14.7 mm to (120.2, 57.5)
- moved A1 7.03 mm to (78.8, 64.5)
- moved D1 1.95 mm to (37.7, 112.4)
- moved D2 1.95 mm to (35.6, 129.4)
- moved D3 1.95 mm to (35.6, 133.7)
- moved H2 1.95 mm to (58.8, 55.8)
- moved H3 1.95 mm to (58.8, 63.0)
- moved H4 1.95 mm to (58.8, 70.2)
- moved J2 1.95 mm to (75.3, 120.8)
- moved JP1 1.95 mm to (37.5, 100.7)
- moved JP3 1.95 mm to (44.9, 110.4)
- moved JP4 1.95 mm to (42.1, 100.7)
- moved R1 1.95 mm to (36.7, 107.1)
- moved RN1 1.95 mm to (30.9, 58.5)
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Other:
- board size 60 x 100 mm -> 100 x 90 mm

Commit message: tmp
Parts:
- moved D2 113.2 mm to (108.1, 42.5)
- moved D3 84.6 mm to (108.8, 91.1), turned to 90 degrees
- moved RN1 80.0 mm to (101.8, 95.6), turned to -90 degrees
- moved JP3 76.1 mm to (86.1, 46.5)
- moved RN3 72.8 mm to (97.8, 95.6), turned to -90 degrees
- moved RN4 72.7 mm to (101.8, 55.0), turned to -90 degrees
- moved D1 71.8 mm to (66.2, 46.5)
- moved R1 71.5 mm to (74.7, 46.5)
- moved RN2 67.3 mm to (97.8, 55.0), turned to -90 degrees
- moved JP1 66.2 mm to (101.8, 84.5), turned to -90 degrees
- moved J1 61.0 mm to (121.8, 118.5), turned to 180 degrees
- moved JP4 58.4 mm to (99.2, 88.5), turned to 90 degrees
- moved J2 55.1 mm to (34.8, 83.5)
- moved H2 51.3 mm to (110.0, 52.6)
- moved H4 50.9 mm to (33.4, 114.3)
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Routing:
- net /SCSI_DATA2: track 0.00 -> 23.9 mm
- net /SCSI_DATA1: track 0.00 -> 23.6 mm
- net /SCSI_DATA3: track 0.00 -> 22.6 mm
- net /SCSI_ATN: track 0.00 -> 22.5 mm
- net /SCSI_DATA0: track 0.00 -> 22.3 mm
- net /SCSI_MSG: track 0.00 -> 21.5 mm
- net /SCSI_ACK: track 0.00 -> 21.5 mm
- net /SCSI_REQ: track 0.00 -> 21.5 mm
- net /SCSI_IO: track 0.00 -> 21.5 mm
- net /SCSI_CD: track 0.00 -> 21.5 mm
- net /SCSI_SEL: track 0.00 -> 21.5 mm
- net /SCSI_RST: track 0.00 -> 21.5 mm
- net /SCSI_BSY: track 0.00 -> 21.5 mm
- net /SCSI_DATA7: track 0.00 -> 21.5 mm
- net /SCSI_DATA6: track 0.00 -> 21.5 mm
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